File: HW/Clock_3LS314A_Atmega328P/BAT_TP4056.kicad_sch (KiCad schematic)
At the start: 19 parts, among them J1 BAT, J2 USB_C_Receptacle_PowerOnly_6P, U2 TP4056-42-ESOP8, U3 DW01A, U4 FS8205A

Commit message: pcb edit
Parts:
- removed J1: BAT, Connector_PinHeader_2.54mm:PinHeader_1x03_P2.54mm_Vertical, symbol Connector:Conn_01x03_Pin
- added J1: Conn_02x02_Counter_Clockwise, Connector_PinHeader_2.00mm:PinHeader_2x02_P2.00mm_Vertical, symbol Connector_Generic:Conn_02x02_Counter_Clockwise
- R6: value 0.2 -> 1
Connections:
- net BAT_VDD: now also J1.1 (Pin_1), J1.4 (Pin_4)
- net at C3.2, U3.6 (GND), U4.1 (S1): now also J1.2 (Pin_2)
- net at R4.1, R5.2, U2.1 (TEMP): now also J1.3 (Pin_3)
Other:
- moved on the sheet: C3
Changed lines of the file:
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@@
+	)
+	(junction
+		(at 176.53 82.55)
+		(diameter 0)
+		(color 0 0 0 0)
 	)
 	(junction
@@
 	(wire
 		(pts
-			(xy 191.77 91.44) (xy 199.39 91.44)
+			(xy 193.04 91.44) (xy 199.39 91.44)
 		)
 		(stroke
@@
 	(wire
 		(pts
-			(xy 191.77 83.82) (xy 199.39 83.82)
+			(xy 193.04 83.82) (xy 199.39 83.82)
 		)
 		(stroke
@@
 	(wire
 		(pts
+			(xy 176.53 80.01) (xy 176.53 82.55)
+		)
+		(stroke
+			(width 0)
+			(type default)
+		)
+	)
+	(wire
+		(pts
 			(xy 105.41 87.63) (xy 115.57 87.63)
 		)
@@
 	(wire
 		(pts
+			(xy 189.23 80.01) (xy 176.53 80.01)
+		)
+		(stroke
+			(width 0)
+			(type default)
+		)
+	)
+	(wire
+		(pts
 			(xy 52.07 95.25) (xy 52.07 113.03)
 		)
@@
 	(wire
 		(pts
+			(xy 189.23 82.55) (xy 189.23 80.01)
+		)
+		(stroke
+			(width 0)
+			(type default)
+		)
+	)
+	(wire
+		(pts
 			(xy 151.13 106.68) (xy 151.13 113.03)
 		)
@@
 	(wire
 		(pts
-			(xy 151.13 87.63) (xy 176.53 87.63)
+			(xy 151.13 87.63) (xy 189.23 87.63)
 		)
 		(stroke
@@
 		(pts
 			(xy 67.31 69.85) (xy 67.31 50.8)
+		)
+		(stroke
+			(width 0)
+			(type default)
+		)
+	)
+	(wire
+		(pts
+			(xy 189.23 85.09) (xy 189.23 87.63)
 		)
 		(stroke
@@
 	(symbol
 		(lib_id "Device:C")
-		(at 191.77 87.63 0)
+		(at 193.04 87.63 0)
 		(unit 1)
 		(exclude_from_sim no)
@@
 		(fields_autoplaced yes)
 		(property "Reference" "C3"
-			(at 195.58 86.3599 0)
+			(at 196.85 86.3599 0)
 			(effects
 				(font
@@
 		)
 		(property "Value" "0.1u"
-			(at 195.58 88.8999 0)
+			(at 196.85 88.8999 0)
 			(effects
 				(font
@@
 		)
 		(property "Footprint" "Capacitor_SMD:C_0603_1608Metric_Pad1.08x0.95mm_HandSolder"
-			(at 192.7352 91.44 0)
+			(at 194.0052 91.44 0)
 			(effects
 				(font
@@
 		)
 		(property "Datasheet" "~"
-			(at 191.77 87.63 0)
+			(at 193.04 87.63 0)
 			(effects
 				(font
@@
 		)
 		(property "Description" "Unpolarized capacitor"
-			(at 191.77 87.63 0)
+			(at 193.04 87.63 0)
 			(effects
 				(font
@@
 			)
 		)
-		(property "Value" "0.2"
+		(property "Value" "1"
 			(at 128.27 59.6899 0)
 			(effects
@@
 	)
 	(symbol
-		(lib_id "Connector:Conn_01x03_Pin")
-		(at 181.61 85.09 0)
-		(mirror y)
+		(lib_id "Connector_Generic:Conn_02x02_Counter_Clockwise")
+		(at 181.61 82.55 0)
 		(unit 1)
 		(exclude_from_sim no)
@@
 		(on_board yes)
 		(dnp no)
+		(fields_autoplaced yes)
 		(property "Reference" "J1"
-			(at 180.975 77.47 0)
-			(effects
-				(font
-					(size 1.27 1.27)
-				)
-			)
-		)
-		(property "Value" "BAT"
-			(at 180.975 80.01 0)
-			(effects
-				(font
-					(size 1.27 1.27)
-				)
-			)
-		)
-		(property "Footprint" "Connector_PinHeader_2.54mm:PinHeader_1x03_P2.54mm_Vertical"
-			(at 181.61 85.09 0)
+			(at 182.88 76.2 0)
+			(effects
+				(font
+					(size 1.27 1.27)
+				)
+			)
+		)
+		(property "Value" "Conn_02x02_Counter_Clockwise"
+			(at 182.88 78.74 0)
+			(effects
+				(font
+					(size 1.27 1.27)
+				)
+			)
+		)
+		(property "Footprint" "Connector_PinHeader_2.00mm:PinHeader_2x02_P2.00mm_Vertical"
+			(at 181.61 82.55 0)
 			(effects
 				(font
@@
 		)
 		(property "Datasheet" "~"
-			(at 181.61 85.09 0)
-			(effects
-				(font
-					(size 1.27 1.27)
-				)
-				(hide yes)
-			)
-		)
-		(property "Description" "Generic connector, single row, 01x03, script generated"
-			(at 181.61 85.09 0)
-			(effects
-				(font
-					(size 1.27 1.27)
-				)
-				(hide yes)
-			)
+			(at 181.61 82.55 0)
+			(effects
+				(font
+					(size 1.27 1.27)
+				)
+				(hide yes)
+			)
+		)
+		(property "Description" "Generic connector, double row, 02x02, counter clockwise pin numbering scheme (similar to DIP package numbering), script generated (kicad-library-utils/schlib/autogen/connector/)"
+			(at 181.61 82.55 0)
+			(effects
+				(font
+					(size 1.27 1.27)
+				)
+				(hide yes)
+			)
+		)
+		(pin "3"
 		)
 		(pin "2"
@@
 		(pin "1"
 		)
-		(pin "3"
+		(pin "4"
 		)
 		(instances

Commit message: pcb edit
Parts:
- added R17, R18, R19, R20: 10k, Resistor_SMD:R_0603_1608Metric_Pad0.98x0.95mm_HandSolder, symbol Device:R
Connections:
- net BAT_GND: now also R17.1, R18.1
- net at C1.1, R1.1, R2.1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: now also U2.8 (CE)
- net at J2.A9 (VBUS), J2.B9 (VBUS), R6.1: now also R19.2, R20.2
- net at J2.A5 (CC1): now also R18.2, R20.1
- net at J2.B5 (CC2): now also R17.2, R19.1
Other:
- moved on the sheet: J2, R7
