File: HW/Clock_3LS314A_Atmega328P/Clock_3LS314A_Atmega328P.kicad_pcb (KiCad board)
At the start: 2 copper layers, 48 parts, among them J1 BAT, J2 USB_C_Receptacle_PowerOnly_6P, J3 AVR_ISP, Q1 BC846, Q2 IRLML5203, Q3 2N7002, Q4 2N7002, Q5 2N7002, Q6 2N7002, SW1 CK_KMS2xxG, U1 ATmega328P-MM, U2 TP4056-42-ESOP8, U3 DW01A, U4 FS8205A, Y1 SJK-7R-32.768-12.5-20-70-C

Commit message: pcb edit
Parts:
- added R15: 15k, Resistor_SMD:R_0603_1608Metric_Pad0.98x0.95mm_HandSolder, B.Cu at (108.0, -45.4)
- added U5: 74LVC1G125, Package_TO_SOT_SMD:SOT-23-5_HandSoldering, B.Cu at (111.3, -45.3)
- C1, C3, C4, C5, C6, C7, C8, C9, J3, Q1, R10, R11, R12, R13, R14, R16, R8, R9, U4, Y1: moved to B.Cu
- J1: value BAT -> Conn_02x02_Counter_Clockwise; footprint Connector_PinHeader_2.54mm:PinHeader_1x03_P2.54mm_Vertical -> Connector_PinHeader_2.00mm:PinHeader_2x02_P2.00mm_Vertical; moved to B.Cu
- Q2: footprint Package_TO_SOT_SMD:SOT-23 -> Package_TO_SOT_SMD:SOT-23_Handsoldering; moved to B.Cu
- R6: value 0.2 -> 1; moved to B.Cu
- moved Q1 62.9 mm to (102.7, -40.0), turned to 180 degrees
- moved R9 58.6 mm to (115.2, -49.4), turned to 180 degrees
- moved R11 55.0 mm to (99.0, -45.5), turned to -90 degrees
- moved R1 54.3 mm to (118.4, -48.7), turned to 180 degrees
- moved R2 54.3 mm to (118.4, -50.3), turned to 180 degrees
- moved R8 53.6 mm to (120.2, -48.5), turned to 180 degrees
- moved R14 52.3 mm to (101.6, -42.8), turned to 180 degrees
- moved C4 51.7 mm to (114.2, -36.1), turned to 180 degrees
- moved C3 51.2 mm to (115.2, -51.0), turned to 180 degrees
- moved R10 50.7 mm to (99.0, -42.0), turned to -90 degrees
- moved R13 48.5 mm to (105.4, -42.8), turned to 180 degrees
- moved R12 48.1 mm to (106.3, -40.1), turned to 90 degrees
- moved C7 43.2 mm to (106.3, -45.5), turned to 90 degrees
- moved Q2 42.3 mm to (102.7, -45.4)
- moved R16 39.5 mm to (114.6, -44.4), turned to -90 degrees
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Connections:
- C4 pad 2: Net-(J3-Pin_4) -> /MCU/MCU_GND
- C5 pad 2: Net-(J3-Pin_4) -> /MCU/MCU_GND
- C6 pad 1: Net-(J3-Pin_4) -> /MCU/MCU_GND
- C8 pad 1: Net-(J3-Pin_4) -> /MCU/MCU_GND
- C9 pad 2: Net-(J3-Pin_4) -> /MCU/MCU_GND
- Q6 pad 3: /MCU/LED1_CAT -> /MCU/LED4_CAT
- RN1 pad 1: /MCU/LED_SegE -> /MCU/LED_SegDot
- RN1 pad 2: /MCU/LED_SegD -> /MCU/LED_SegC
- RN1 pad 3: /MCU/LED_SegC -> /MCU/LED_SegD
- RN1 pad 4: /MCU/LED_SegDot -> /MCU/LED_SegE
- RN1 pad 6: Net-(RN1-R3.2) -> /MCU/KEY_IRQ
- RN2 pad 1: /MCU/LED_SegB -> /MCU/LED_SegF
- RN2 pad 2: /MCU/LED_SegA -> /MCU/LED_SegG
- RN2 pad 3: /MCU/LED_SegG -> /MCU/LED_SegA
- RN2 pad 4: /MCU/LED_SegF -> /MCU/LED_SegB
- RN3 pad 1: /MCU/LED_DRIVE_4 -> /MCU/MCU_LED_DRIVE_4
- RN3 pad 2: /MCU/LED_DRIVE_3 -> /MCU/MCU_LED_DRIVE_3
- RN3 pad 3: /MCU/LED_DRIVE_2 -> /MCU/MCU_LED_DRIVE_2
- RN3 pad 4: /MCU/LED_DRIVE_1 -> /MCU/MCU_LED_DRIVE_1
- RN3 pad 5: /MCU/MCU_LED_DRIVE_1 -> /MCU/LED_DRIVE_1
- RN3 pad 6: /MCU/MCU_LED_DRIVE_2 -> /MCU/LED_DRIVE_2
- RN3 pad 7: /MCU/MCU_LED_DRIVE_3 -> /MCU/LED_DRIVE_3
- RN3 pad 8: /MCU/MCU_LED_DRIVE_4 -> /MCU/LED_DRIVE_4
- SW1 pad 2: /MCU/MCU_VDD -> Net-(R15-Pad2)
- U1 pad 1: Net-(RN1-R1.2) -> Net-(RN1-R4.2)
- U1 pad 12: unconnected-(U1-PB2-Pad12) -> /MCU/KEY_OFF
- U1 pad 2: Net-(RN2-R4.2) -> Net-(RN2-R1.2)
- U1 pad 24: Net-(RN1-R2.2) -> /MCU/MCU_KEY_1
- U1 pad 26: Net-(RN1-R4.2) -> Net-(RN1-R1.2)
- U1 pad 27: Net-(RN1-R3.2) -> Net-(RN1-R2.2)
- U1 pad 28: /MCU/MCU_KEY_1 -> /MCU/KEY_IRQ
- U1 pad 7: Net-(RN2-R3.2) -> Net-(RN2-R2.2)
- U1 pad 8: Net-(RN2-R2.2) -> Net-(RN2-R3.2)
- U1 pad 9: Net-(RN2-R1.2) -> Net-(RN2-R4.2)
Routing:
- net /MCU/MCU_KEY_1: track 0.00 -> 48.8 mm, vias 0 -> 3
- net /MCU/LED_SegG: track 0.00 -> 40.8 mm, vias 0 -> 5
- net /MCU/LED_SegF: track 0.00 -> 39.9 mm, vias 0 -> 1
- net /MCU/MCU_VDD: track 0.00 -> 38.9 mm, vias 0 -> 17
- net /MCU/MCU_VBAT_CONTROL: track 0.00 -> 37.8 mm, vias 0 -> 2
- net Net-(U2-V_{CC}): track 0.00 -> 36.8 mm, vias 0 -> 3
- net /MCU/LED_SegD: track 0.00 -> 34.9 mm
- net /MCU/LED_SegB: track 0.00 -> 31.3 mm, vias 0 -> 1
- net /MCU/LED4_CAT: track 0.00 -> 30.7 mm, vias 0 -> 2
- net /MCU/LED_SegA: track 0.00 -> 30.3 mm, vias 0 -> 4
- net /MCU/LED_DRIVE_1: track 0.00 -> 29.2 mm, vias 0 -> 2
- net /MCU/LED_SegDot: track 0.00 -> 29.0 mm, vias 0 -> 4
- net Net-(R15-Pad2): track 0.00 -> 28.2 mm, vias 0 -> 2
- net /MCU/LED_DRIVE_3: track 0.00 -> 28.0 mm, vias 0 -> 2
- net /MCU/LED_SegE: track 0.00 -> 27.0 mm, vias 0 -> 2
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- added copper zone on B.Cu, net /MCU/MCU_GND
- added copper zone on F.Cu, net /MCU/MCU_GND
- added copper zone on In2.Cu, net /MCU/MCU_GND
- added copper zone on In1.Cu, net /MCU/MCU_VDD
- added copper zone on In2.Cu, net /MCU/MCU_VDD
Other:
- board outline added: 41 x 23.5 mm
- copper layers 2 -> 4

Commit message: pcb edit
Parts:
- added R17: 10k, Resistor_SMD:R_0603_1608Metric_Pad0.98x0.95mm_HandSolder, B.Cu at (91.8, -42.1)
- added R18: 10k, Resistor_SMD:R_0603_1608Metric_Pad0.98x0.95mm_HandSolder, B.Cu at (93.4, -42.1)
- added R19: 10k, Resistor_SMD:R_0603_1608Metric_Pad0.98x0.95mm_HandSolder, B.Cu at (96.5, -33.2)
- added R20: 10k, Resistor_SMD:R_0603_1608Metric_Pad0.98x0.95mm_HandSolder, B.Cu at (98.0, -33.2)
- moved Y1 1.45 mm to (114.3, -39.0)
- moved C8 1.42 mm to (111.7, -38.2)
- moved C9 1.41 mm to (111.7, -39.8)
Connections:
- C1 pad 1: Net-(U2-V_{CC}) -> Net-(U2-CE)
- J2 pad A5: unconnected-(J2-CC1-PadA5) -> Net-(J2-CC1)
- J2 pad B5: unconnected-(J2-CC2-PadB5) -> Net-(J2-CC2)
- R1 pad 1: Net-(U2-V_{CC}) -> Net-(U2-CE)
- R2 pad 1: Net-(U2-V_{CC}) -> Net-(U2-CE)
- R4 pad 2: Net-(U2-V_{CC}) -> Net-(U2-CE)
- R6 pad 2: Net-(U2-V_{CC}) -> Net-(U2-CE)
- U2 pad 4: Net-(U2-V_{CC}) -> Net-(U2-CE)
- U2 pad 8: unconnected-(U2-CE-Pad8) -> Net-(U2-CE)
Routing:
- net Net-(U2-CE): track 0.00 -> 41.3 mm, vias 0 -> 4
- net Net-(U2-V_{CC}): track 36.8 -> 0.00 mm, vias 3 -> 0
- net /MCU/LED_SegC: track 20.5 -> 39.6 mm
- net Net-(J2-CC2): track 0.00 -> 15.7 mm, vias 0 -> 1
- net Net-(J2-CC1): track 0.00 -> 13.3 mm, vias 0 -> 1
- net /MCU/LED_SegDot: track 29.0 -> 38.3 mm
- net Net-(J2-VBUS-PadA9): track 16.9 -> 26.3 mm, vias 1 -> 2
- net Net-(U3-VCC): track 0.00 -> 3.90 mm
- net /MCU/MCU_VDD: track 38.9 -> 41.8 mm, vias 17 -> 11
- net /MCU/MCU_GND: track 12.8 -> 10.2 mm, vias 4 -> 16
- net Net-(U1-XTAL1/PB6): track 4.29 -> 6.17 mm
- net Net-(U1-XTAL2/PB7): track 4.23 -> 6.06 mm
- net Net-(J1-Pin_3): track 15.2 -> 15.9 mm
- net /MCU/MCU_VBAT_CONTROL: track 37.8 -> 37.3 mm
- added copper zone on In1.Cu, net /MCU/MCU_GND
- removed copper zone on In2.Cu, net /MCU/MCU_VDD
Other:
- outline, holes or cut-outs redrawn
- board text added: "2026"
- board text added: "2L314 Clock"
- board text added: "maxssau"
- board text added: "v0.1"
